Commit message: rename links and joints

File: urdf/MAGICBOT_with_hand.urdf (robot description, URDF)
Before this commit: robot Magicbot-Gen1, 58 links, 57 joints
Links:
- removed link LINK_ANKLE_PITCH_L
- removed link LINK_ANKLE_PITCH_R
- removed link LINK_ANKLE_ROLL_L
- removed link LINK_ANKLE_ROLL_R
- removed link LINK_HIP_PITCH_L
- removed link LINK_HIP_PITCH_R
- removed link LINK_HIP_ROLL_L
- removed link LINK_HIP_ROLL_R
- removed link LINK_HIP_YAW_L
- removed link LINK_HIP_YAW_R
- removed link LINK_KNEE_PITCH_L
- removed link LINK_KNEE_PITCH_R
- removed link link_hp
- removed link link_hy
- removed link link_la1
- removed link link_la2
- removed link link_la3
- removed link link_la4
- removed link link_la5
- removed link link_la6
- removed link link_ra1
- removed link link_ra2
- removed link link_ra3
- removed link link_ra4
- removed link link_ra5
- removed link link_ra6
- removed link link_wr
- removed link link_wy
- added link head_pitch_link, mass 1.75103035; collision mesh filename=package://magicbot-gen1_description/meshes/head_pitch_link.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; visual mesh filename=package://magicbot-gen1_description/meshes/head_pitch_link.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
- added link head_yaw_link, mass 1.30579318; collision mesh filename=package://magicbot-gen1_description/meshes/head_yaw_link.STL; visual mesh filename=package://magicbot-gen1_description/meshes/head_yaw_link.STL
- added link left_ankle_pitch_link, mass 0.0724143; collision mesh filename=package://magicbot-gen1_description/meshes/left_ankle_pitch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; visual mesh filename=package://magicbot-gen1_description/meshes/left_ankle_pitch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
- added link left_ankle_roll_link, mass 0.80130806; collision mesh filename=package://magicbot-gen1_description/meshes/left_ankle_roll_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; visual mesh filename=package://magicbot-gen1_description/meshes/left_ankle_roll_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
- added link left_elbow_roll_link, mass 0.17421; collision mesh filename=package://magicbot-gen1_description/meshes/left_elbow_roll_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; visual mesh filename=package://magicbot-gen1_description/meshes/left_elbow_roll_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
- added link left_hip_pitch_link, mass 5.04878347; collision mesh filename=package://magicbot-gen1_description/meshes/left_hip_pitch_l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; visual mesh filename=package://magicbot-gen1_description/meshes/left_hip_pitch_l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
- added link left_hip_roll_link, mass 0.47382; collision mesh filename=package://magicbot-gen1_description/meshes/left_hip_roll_li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; visual mesh filename=package://magicbot-gen1_description/meshes/left_hip_roll_li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
- added link left_hip_yaw_link, mass 3.3831774; collision mesh filename=package://magicbot-gen1_description/meshes/left_hip_yaw_lin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; visual mesh filename=package://magicbot-gen1_description/meshes/left_hip_yaw_lin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
- added link left_knee_pitch_link, mass 3.37617301; collision mesh filename=package://magicbot-gen1_description/meshes/left_knee_pitch_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; visual mesh filename=package://magicbot-gen1_description/meshes/left_knee_pitch_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
- added link left_shoulder_pitch_link, mass 1.4531; collision mesh filename=package://magicbot-gen1_description/meshes/left_shoulder_pi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; visual mesh filename=package://magicbot-gen1_description/meshes/left_shoulder_pi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
- added link left_shoulder_roll_link, mass 0.53748; collision mesh filename=package://magicbot-gen1_description/meshes/left_shoulder_ro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; visual mesh filename=package://magicbot-gen1_description/meshes/left_shoulder_ro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
- added link left_shoulder_yaw_link, mass 1.784; collision mesh filename=package://magicbot-gen1_description/meshes/left_shoulder_ya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; visual mesh filename=package://magicbot-gen1_description/meshes/left_shoulder_ya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
- added link left_wrist_roll_link, mass 0.022425; collision mesh filename=package://magicbot-gen1_description/meshes/left_wrist_roll_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; visual mesh filename=package://magicbot-gen1_description/meshes/left_wrist_roll_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
- added link left_wrist_yaw_link, mass 1.9293; collision mesh filename=package://magicbot-gen1_description/meshes/left_wrist_yaw_l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; visual mesh filename=package://magicbot-gen1_description/meshes/left_wrist_yaw_l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
- added link right_ankle_pitch_link, mass 0.0724143; collision mesh filename=package://magicbot-gen1_description/meshes/right_ankle_pitc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; visual mesh filename=package://magicbot-gen1_description/meshes/right_ankle_pitc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
- added link right_ankle_roll_link, mass 0.79424534; collision mesh filename=package://magicbot-gen1_description/meshes/right_ankle_roll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; visual mesh filename=package://magicbot-gen1_description/meshes/right_ankle_roll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
- added link right_elbow_roll_link, mass 0.17421; collision mesh filename=package://magicbot-gen1_description/meshes/right_elbow_roll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; visual mesh filename=package://magicbot-gen1_description/meshes/right_elbow_roll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
- added link right_hip_pitch_link, mass 5.04801978; collision mesh filename=package://magicbot-gen1_description/meshes/right_hip_pitch_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; visual mesh filename=package://magicbot-gen1_description/meshes/right_hip_pitch_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
- added link right_hip_roll_link, mass 0.47383286; collision mesh filename=package://magicbot-gen1_description/meshes/right_hip_roll_l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; visual mesh filename=package://magicbot-gen1_description/meshes/right_hip_roll_l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
- added link right_hip_yaw_link, mass 3.38317107; collision mesh filename=package://magicbot-gen1_description/meshes/right_hip_yaw_li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; visual mesh filename=package://magicbot-gen1_description/meshes/right_hip_yaw_li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
- added link right_knee_pitch_link, mass 3.37418513; collision mesh filename=package://magicbot-gen1_description/meshes/right_knee_pitch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; visual mesh filename=package://magicbot-gen1_description/meshes/right_knee_pitch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
- added link right_shoulder_pitch_link, mass 1.4531; collision mesh filename=package://magicbot-gen1_description/meshes/right_shoulder_p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; visual mesh filename=package://magicbot-gen1_description/meshes/right_shoulder_p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
- added link right_shoulder_roll_link, mass 0.53748; collision mesh filename=package://magicbot-gen1_description/meshes/right_shoulder_r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; visual mesh filename=package://magicbot-gen1_description/meshes/right_shoulder_r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
- added link right_shoulder_yaw_link, mass 1.784; collision mesh filename=package://magicbot-gen1_description/meshes/right_shoulder_y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; visual mesh filename=package://magicbot-gen1_description/meshes/right_shoulder_y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
- added link right_wrist_roll_link, mass 0.022425; collision mesh filename=package://magicbot-gen1_description/meshes/right_wrist_roll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; visual mesh filename=package://magicbot-gen1_description/meshes/right_wrist_roll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
- added link right_wrist_yaw_link, mass 1.9293; collision mesh filename=package://magicbot-gen1_description/meshes/right_wrist_yaw_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; visual mesh filename=package://magicbot-gen1_description/meshes/right_wrist_yaw_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
- added link waist_roll_link, mass 2.52447836; collision mesh filename=package://magicbot-gen1_description/meshes/waist_roll_link.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; visual mesh filename=package://magicbot-gen1_description/meshes/waist_roll_link.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
- added link waist_yaw_link, mass 15.00776677; collision mesh filename=package://magicbot-gen1_description/meshes/waist_yaw_link.S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; visual mesh filename=package://magicbot-gen1_description/meshes/waist_yaw_link.S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
Joints:
- removed joint JOINT_ANKLE_PITCH_L
- removed joint JOINT_ANKLE_PITCH_R
- removed joint JOINT_ANKLE_ROLL_L
- removed joint JOINT_ANKLE_ROLL_R
- removed joint JOINT_HIP_PITCH_L
- removed joint JOINT_HIP_PITCH_R
- removed joint JOINT_HIP_ROLL_L
- removed joint JOINT_HIP_ROLL_R
- removed joint JOINT_HIP_YAW_L
- removed joint JOINT_HIP_YAW_R
- removed joint JOINT_KNEE_PITCH_L
- removed joint JOINT_KNEE_PITCH_R
- removed joint joint_hp
- removed joint joint_hy
- removed joint joint_la1
- removed joint joint_la2
- removed joint joint_la3
- removed joint joint_la4
- removed joint joint_la5
- removed joint joint_la6
- removed joint joint_la7
- removed joint joint_ra1
- removed joint joint_ra2
- removed joint joint_ra3
- removed joint joint_ra4
- removed joint joint_ra5
- removed joint joint_ra6
- removed joint joint_ra7
- removed joint joint_wr
- removed joint joint_wy
- added joint head_pitch_joint: type revolute, parent head_yaw_link, child head_pitch_link, origin xyz=-0.0065 2.3658E-05 0 rpy=0 0 0, axis 0 1 0, limit lower=-0.349 upper=0.349 effort=60 velocity=15
- added joint head_yaw_joint: type revolute, parent waist_yaw_link, child head_yaw_link, origin xyz=-0.0059657 0 0.50108 rpy=0 0 0, axis 0 0 1, limit lower=-1.047 upper=1.047 effort=60 velocity=15
- added joint left_ankle_pitch_joint: type revolute, parent left_knee_pitch_link, child left_ankle_pitch_link, origin xyz=0.035056 0 -0.3867 rpy=0 0 0, axis 0 1 0, limit lower=-1.308 upper=0.523 effort=120 velocity=15
- added joint left_ankle_roll_joint: type revolute, parent left_ankle_pitch_link, child left_ankle_roll_link, origin xyz=0 0 -0.01 rpy=0 0 0, axis 1 0 0, limit lower=-0.349 upper=0.349 effort=120 velocity=15
- added joint left_elbow_roll_joint: type revolute, parent left_shoulder_yaw_link, child left_elbow_roll_link, origin xyz=-0.00074295 -0.0049956 -0.15199 rpy=-0.00018277 0.0001556 -4.8773E-05, axis 1 0 0, limit lower=-2.215 upper=0.174 effort=100 velocity=5
- added joint left_hip_pitch_joint: type revolute, parent left_hip_yaw_link, child left_hip_pitch_link, origin xyz=0 0 -0.118 rpy=0 0 0, axis 0 1 0, limit lower=-2.093 upper=0.698 effort=360 velocity=15
- added joint left_hip_roll_joint: type revolute, parent pelvis, child left_hip_roll_link, origin xyz=0 0.1175 0 rpy=0 0 0, axis 1 0 0, limit lower=-0.349 upper=0.523 effort=360 velocity=15
- added joint left_hip_yaw_joint: type revolute, parent left_hip_roll_link, child left_hip_yaw_link, origin xyz=0 0 0 rpy=0 0 0, axis 0 0 1, limit lower=-0.262 upper=0.523 effort=60 velocity=15
- added joint left_knee_pitch_joint: type revolute, parent left_hip_pitch_link, child left_knee_pitch_link, origin xyz=-0.03295 0 -0.3875 rpy=0 0 0, axis 0 1 0, limit lower=0 upper=2.617 effort=360 velocity=15
- added joint left_shoulder_pitch_joint: type revolute, parent waist_yaw_link, child left_shoulder_pitch_link, origin xyz=-0.0078982 0.19799 0.346 rpy=0 0 0, axis 0 1 0, limit lower=-2.756 upper=2.756 effort=110 velocity=5
- added joint left_shoulder_roll_joint: type revolute, parent left_shoulder_pitch_link, child left_shoulder_roll_link, origin xyz=0 0 0 rpy=0 0 0, axis 1 0 0, limit lower=-0.262 upper=2.878 effort=110 velocity=5
- added joint left_shoulder_yaw_joint: type revolute, parent left_shoulder_roll_link, child left_shoulder_yaw_link, origin xyz=0 0.015686 -0.10553 rpy=0.087267 0 0, axis 0 0 1, limit lower=-2.617 upper=2.617 effort=100 velocity=5
- added joint left_wrist_pitch_joint: type revolute, parent left_wrist_roll_link, child hand_link, origin xyz=0 0 0 rpy=0 0 0, axis 0 1 0, limit lower=-0.857 upper=1.2036 effort=0 velocity=0
- added joint left_wrist_roll_joint: type revolute, parent left_wrist_yaw_link, child left_wrist_roll_link, origin xyz=0 0.02371 -0.29785 rpy=0 0 0, axis 1 0 0, limit lower=-1.099 upper=0.855 effort=40 velocity=5
- added joint left_wrist_yaw_joint: type revolute, parent left_elbow_roll_link, child left_wrist_yaw_link, origin xyz=0 0 0 rpy=0 0 0, axis 0 0 1, limit lower=-2.913 upper=2.913 effort=100 velocity=5
- added joint right_ankle_pitch_joint: type revolute, parent right_knee_pitch_link, child right_ankle_pitch_link, origin xyz=0.035003 0 -0.3867 rpy=0 0 0, axis 0 1 0, limit lower=-1.308 upper=0.523 effort=120 velocity=15
- added joint right_ankle_roll_joint: type revolute, parent right_ankle_pitch_link, child right_ankle_roll_link, origin xyz=0 0 -0.01 rpy=4.0892E-05 0.00014855 0, axis 1 0 0, limit lower=-0.349 upper=0.349 effort=120 velocity=15
- added joint right_elbow_roll_joint: type revolute, parent right_shoulder_yaw_link, child right_elbow_roll_link, origin xyz=0.00074295 0.0049956 -0.15199 rpy=0.00018277 -0.0001556 -4.8773E-05, axis 1 0 0, limit lower=-0.174 upper=2.215 effort=100 velocity=5
- added joint right_hip_pitch_joint: type revolute, parent right_hip_yaw_link, child right_hip_pitch_link, origin xyz=0 0 -0.118 rpy=0 0 0, axis 0 1 0, limit lower=-2.093 upper=0.698 effort=360 velocity=15
- added joint right_hip_roll_joint: type revolute, parent pelvis, child right_hip_roll_link, origin xyz=0 -0.1175 0 rpy=0 0 0, axis 1 0 0, limit lower=-0.523 upper=0.349 effort=360 velocity=15
- added joint right_hip_yaw_joint: type revolute, parent right_hip_roll_link, child right_hip_yaw_link, origin xyz=0 0 0 rpy=0 0 0, axis 0 0 1, limit lower=-0.523 upper=0.262 effort=60 velocity=15
- added joint right_knee_pitch_joint: type revolute, parent right_hip_pitch_link, child right_knee_pitch_link, origin xyz=-0.032951 0 -0.3875 rpy=0 0 0, axis 0 1 0, limit lower=0 upper=2.617 effort=360 velocity=15
- added joint right_shoulder_pitch_joint: type revolute, parent waist_yaw_link, child right_shoulder_pitch_link, origin xyz=-0.0079 -0.198 0.346 rpy=0 0 0, axis 0 1 0, limit lower=-2.756 upper=2.756 effort=110 velocity=5
- added joint right_shoulder_roll_joint: type revolute, parent right_shoulder_pitch_link, child right_shoulder_roll_link, origin xyz=0 0 0 rpy=0 0 0, axis 1 0 0, limit lower=-2.878 upper=0.262 effort=110 velocity=5
- added joint right_shoulder_yaw_joint: type revolute, parent right_shoulder_roll_link, child right_shoulder_yaw_link, origin xyz=1.2039E-05 -0.015686 -0.10553 rpy=-0.087267 0 0, axis 0 0 1, limit lower=-2.617 upper=2.617 effort=100 velocity=5
- added joint right_wrist_pitch_joint: type revolute, parent right_wrist_roll_link, child hand_Link_R, origin xyz=0 0 0 rpy=0 0 0, axis 0 1 0, limit lower=-1.2036 upper=0.857 effort=0 velocity=0
- added joint right_wrist_roll_joint: type revolute, parent right_wrist_yaw_link, child right_wrist_roll_link, origin xyz=0 -0.02371 -0.29785 rpy=0 0 0, axis 1 0 0, limit lower=-0.855 upper=1.099 effort=40 velocity=5
- added joint right_wrist_yaw_joint: type revolute, parent right_elbow_roll_link, child right_wrist_yaw_link, origin xyz=0 0 0 rpy=0 0 0, axis 0 0 1, limit lower=-2.913 upper=2.913 effort=100 velocity=5
- added joint waist_roll_joint: type revolute, parent pelvis, child waist_roll_link, origin xyz=-0.016 0 0.083 rpy=0 0 0, axis 1 0 0, limit lower=-0.349 upper=0.349 effort=200 velocity=5
- added joint waist_yaw_joint: type revolute, parent waist_roll_link, child waist_yaw_link, origin xyz=0 0 0 rpy=0 0 0, axis 0 0 1, limit lower=-1.57 upper=1.57 effort=100 velocity=5
- joint joint_head_rgb_f: parent link_hp -> head_pitch_link
- joint joint_head_rgbd: parent link_hp -> head_pitch_link
- joint logo_joint: parent link_wy -> waist_yaw_link

Commit message: Update joint limits

File: urdf/MAGICBOT.urdf (robot description, URDF)
Before this commit: robot Magicbot-Gen1, 36 links, 35 joints
Joints:
- joint left_elbow_roll_joint: limit lower=-2.215 upper=0.174 effort=100 velocity=5 -> lower=-2.079 upper=0.035 effort=100 velocity=5
- joint left_shoulder_pitch_joint: limit lower=-2.756 upper=2.756 effort=110 velocity=5 -> lower=-2.619 upper=2.619 effort=110 velocity=5
- joint left_shoulder_roll_joint: limit lower=-0.262 upper=2.878 effort=110 velocity=5 -> lower=-0.122 upper=2.739 effort=110 velocity=5
- joint left_shoulder_yaw_joint: limit lower=-2.617 upper=2.617 effort=100 velocity=5 -> lower=-2.478 upper=2.478 effort=100 velocity=5
- joint left_wrist_pitch_joint: limit lower=-0.454 upper=0.454 effort=40 velocity=5 -> lower=-0.314 upper=0.314 effort=40 velocity=5
- joint left_wrist_roll_joint: limit lower=-1.099 upper=0.855 effort=40 velocity=5 -> lower=-0.959 upper=0.715 effort=40 velocity=5
- joint left_wrist_yaw_joint: limit lower=-2.913 upper=2.913 effort=100 velocity=5 -> lower=-2.744 upper=2.744 effort=100 velocity=5
- joint right_elbow_roll_joint: limit lower=-0.174 upper=2.215 effort=100 velocity=5 -> lower=-0.035 upper=2.079 effort=100 velocity=5
- joint right_shoulder_pitch_joint: limit lower=-2.756 upper=2.756 effort=110 velocity=5 -> lower=-2.619 upper=2.619 effort=110 velocity=5
- joint right_shoulder_roll_joint: limit lower=-2.878 upper=0.262 effort=110 velocity=5 -> lower=-2.739 upper=0.122 effort=110 velocity=5
- joint right_shoulder_yaw_joint: limit lower=-2.617 upper=2.617 effort=100 velocity=5 -> lower=-2.478 upper=2.478 effort=100 velocity=5
- joint right_wrist_pitch_joint: limit lower=-0.454 upper=0.454 effort=40 velocity=5 -> lower=-0.314 upper=0.314 effort=40 velocity=5
- joint right_wrist_roll_joint: limit lower=-0.855 upper=1.099 effort=40 velocity=5 -> lower=-0.715 upper=0.959 effort=40 velocity=5
- joint right_wrist_yaw_joint: limit lower=-2.913 upper=2.913 effort=100 velocity=5 -> lower=-2.744 upper=2.744 effort=100 velocity=5

File: urdf/MAGICBOT_with_hand.urdf (robot description, URDF)
Before this commit: robot Magicbot-Gen1, 58 links, 57 joints
Joints:
- joint left_elbow_roll_joint: limit lower=-2.215 upper=0.174 effort=100 velocity=5 -> lower=-2.079 upper=0.035 effort=100 velocity=5
- joint left_shoulder_pitch_joint: limit lower=-2.756 upper=2.756 effort=110 velocity=5 -> lower=-2.619 upper=2.619 effort=110 velocity=5
- joint left_shoulder_roll_joint: limit lower=-0.262 upper=2.878 effort=110 velocity=5 -> lower=-0.122 upper=2.739 effort=110 velocity=5
- joint left_shoulder_yaw_joint: limit lower=-2.617 upper=2.617 effort=100 velocity=5 -> lower=-2.478 upper=2.478 effort=100 velocity=5
- joint left_wrist_pitch_joint: limit lower=-0.857 upper=1.2036 effort=0 velocity=0 -> lower=-0.314 upper=0.314 effort=40 velocity=5
- joint left_wrist_roll_joint: limit lower=-1.099 upper=0.855 effort=40 velocity=5 -> lower=-0.959 upper=0.715 effort=40 velocity=5
- joint left_wrist_yaw_joint: limit lower=-2.913 upper=2.913 effort=100 velocity=5 -> lower=-2.744 upper=2.744 effort=100 velocity=5
- joint right_elbow_roll_joint: limit lower=-0.174 upper=2.215 effort=100 velocity=5 -> lower=-0.035 upper=2.079 effort=100 velocity=5
- joint right_shoulder_pitch_joint: limit lower=-2.756 upper=2.756 effort=110 velocity=5 -> lower=-2.619 upper=2.619 effort=110 velocity=5
- joint right_shoulder_roll_joint: limit lower=-2.878 upper=0.262 effort=110 velocity=5 -> lower=-2.739 upper=0.122 effort=110 velocity=5
- joint right_shoulder_yaw_joint: limit lower=-2.617 upper=2.617 effort=100 velocity=5 -> lower=-2.478 upper=2.478 effort=100 velocity=5
- joint right_wrist_pitch_joint: limit lower=-1.2036 upper=0.857 effort=0 velocity=0 -> lower=-0.314 upper=0.314 effort=0 velocity=0
- joint right_wrist_roll_joint: limit lower=-0.855 upper=1.099 effort=40 velocity=5 -> lower=-0.715 upper=0.959 effort=40 velocity=5
- joint right_wrist_yaw_joint: limit lower=-2.913 upper=2.913 effort=100 velocity=5 -> lower=-2.744 upper=2.744 effort=100 velocity=5
